Commit message: Gazebo plugins working

File: description/inertial.macros.xacro (robot description, xacro)
@@ -21,3 +21,12 @@
         </inertial>
     </xacro:macro>
+    <xacro:macro name="inertial_sphere" params="mass radius *origin">
+        <inertial>
+            <xacro:insert_block name="origin"/>
+            <mass value="${mass}" />
+            <inertia ixx="${(2/5) * mass * radius * radius}" ixy="0.0" ixz="0.0"
+                    iyy="${(2/5) * mass * radius * radius}" iyz="0.0"
+                    izz="${(2/5) * mass * radius * radius}" />
+        </inertial>
+    </xacro:macro>
 </robot>

File: description/robot.body.xacro (robot description, xacro)
@@ -75,6 +75,6 @@
         <parent link="base_link"/>
         <child link="rear_right_wheel"/>
-        <origin xyz="-0.2 -0.175 0" rpy="-${pi/2} 0 0"/>
-        <axis xyz="0 0 1"/>
+        <origin xyz="-0.2 -0.175 0" rpy="${pi/2} 0 0"/>
+        <axis xyz="0 0 -1"/>
     </joint>
     <link name="rear_right_wheel">
@@ -104,19 +104,24 @@
     <link name="caster">
         <visual>
-            <origin xyz="0.05 0 0.05"/>
+            <origin xyz="0.05 0 0"/>
             <geometry>
-                <sphere radius="0.05"/>
+                <sphere radius="0.1"/>
             </geometry>
             <material name="red"/>
         </visual>
         <collision>
-            <origin xyz="0.05 0 0.05"/>
+            <origin xyz="0.05 0 0"/>
             <geometry>
-                <cylinder radius="0.05" length="0.02"/>
+                <sphere radius="0.1"/>
             </geometry>
         </collision>
-        <xacro:inertial_cylinder mass="0.05" length="0.02" radius="0.05">
-            <origin xyz="0.05 0 0.05" rpy="0 0 0"/>
-        </xacro:inertial_cylinder>
+        <xacro:inertial_sphere mass="0.1" radius="0.1">
+            <origin xyz="0.05 0 0" rpy="0 0 0"/>
+        </xacro:inertial_sphere>
     </link>
+    <gazebo reference="caster">
+        <material>Gazebo/Red</material>
+        <mu1 value="0.01"/>
+        <mu2 value="0.01"/>
+    </gazebo>
 </robot>
